File: KiCad/tu9Replacement.kicad_sch (KiCad schematic)
At the start: 24 parts, among them J1 Conn_01x10

Commit message: parity with local work
Parts:
- removed RV1, RV2: 100k, symbol Device:R_POT_Small
- added RV? (x2): 100k, symbol Device:R_Potentiometer_Small
- C1: value 10n -> 10nF
- C2: value 1u -> 1uF
Connections:
- net +5V: now also RV?.3
- net GND: now also RV?.1, RV?.3
- net sine: now also RV?.1
- net at C2.2, R4.1: now also RV?.2
- net at C1.2: now also RV?.2
Other:
- note added: "Everything after the ${00000000-0000-0000-0000-00006156584c:VALUE} cap is unnecessary for the ts-811a, but I'll leave it in case another radio does need it"
- company: jared -> jared jackson
- title: te-9 -> tu-5 Replacement
Changed lines of the file:
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@@
   (paper "A4")
   (title_block
-    (title "te-9")
+    (title "tu-5 Replacement")
     (date "2021-09-24")
     (rev "v1")
-    (company "jared")
+    (company "jared jackson")
     (comment 1 "ctcss tone encoder for kenwood ts-811a")
   )
@@
   (text "just so erc wont yell" (at 101.6 102.87 180)
     (effects (font (size 1.27 1.27)) (justify right bottom))
+  )
+  (text "Everything after the ${00000000-0000-0000-0000-00006156584c:VALUE} cap is\nunnecessary for the ts-811a, but\nI'll leave it in case another\nradio does need it"
+    (at 224.79 83.82 0)
+    (effects (font (size 1.27 1.27)) (justify left bottom))
   )
   (text "connector to radio" (at 101.6 60.96 180)
@@
     (pin "2")
   )
-  (symbol (lib_id "Device:R_POT_Small") (at 191.77 68.58 0) (unit 1)
-    (in_bom yes) (on_board yes)
-    (property "Reference" "RV1" (id 0) (at 190.2714 67.4116 0)
-      (effects (font (size 1.27 1.27)) (justify right))
-    )
-    (property "Value" "100k" (id 1) (at 190.2714 69.723 0)
-      (effects (font (size 1.27 1.27)) (justify right))
-    )
-    (property "Footprint" "" (id 2) (at 191.77 68.58 0)
-      (effects (font (size 1.27 1.27)) hide)
-    )
-    (property "Datasheet" "~" (id 3) (at 191.77 68.58 0)
-      (effects (font (size 1.27 1.27)) hide)
-    )
-    (pin "1")
-    (pin "2")
-    (pin "3")
-  )
-  (symbol (lib_id "Device:R_POT_Small") (at 217.17 80.01 0) (mirror y) (unit 1)
-    (in_bom yes) (on_board yes)
-    (property "Reference" "RV2" (id 0) (at 218.6686 78.8416 0)
-      (effects (font (size 1.27 1.27)) (justify right))
-    )
-    (property "Value" "100k" (id 1) (at 218.6686 81.153 0)
-      (effects (font (size 1.27 1.27)) (justify right))
-    )
-    (property "Footprint" "" (id 2) (at 217.17 80.01 0)
-      (effects (font (size 1.27 1.27)) hide)
-    )
-    (property "Datasheet" "~" (id 3) (at 217.17 80.01 0)
-      (effects (font (size 1.27 1.27)) hide)
-    )
-    (pin "1")
-    (pin "2")
-    (pin "3")
-  )
   (symbol (lib_id "Device:C_Small") (at 199.39 68.58 270) (unit 1)
     (in_bom yes) (on_board yes)
     (property "Reference" "C1" (id 0) (at 199.39 62.7634 90))
-    (property "Value" "10n" (id 1) (at 199.39 65.0748 90))
+    (property "Value" "10nF" (id 1) (at 199.39 65.0748 90))
     (property "Footprint" "" (id 2) (at 199.39 68.58 0)
       (effects (font (size 1.27 1.27)) hide)
@@
       (effects (font (size 1.27 1.27)) (justify right))
     )
-    (property "Value" "1u" (id 1) (at 208.0768 81.153 0)
+    (property "Value" "1uF" (id 1) (at 208.0768 81.153 0)
       (effects (font (size 1.27 1.27)) (justify right))
     )
@@
     )
     (pin "1")
+  )
+  (symbol (lib_id "Device:R_Potentiometer_Small") (at 191.77 68.58 0) (unit 1)
+    (in_bom yes) (on_board yes) (fields_autoplaced)
+    (property "Reference" "RV?" (id 0) (at 190.2461 67.6715 0)
+      (effects (font (size 1.27 1.27)) (justify right))
+    )
+    (property "Value" "100k" (id 1) (at 190.2461 70.4466 0)
+      (effects (font (size 1.27 1.27)) (justify right))
+    )
+    (property "Footprint" "" (id 2) (at 191.77 68.58 0)
+      (effects (font (size 1.27 1.27)) hide)
+    )
+    (property "Datasheet" "~" (id 3) (at 191.77 68.58 0)
+      (effects (font (size 1.27 1.27)) hide)
+    )
+    (pin "1")
+    (pin "2")
+    (pin "3")
+  )
+  (symbol (lib_id "Device:R_Potentiometer_Small") (at 217.17 80.01 180) (unit 1)
+    (in_bom yes) (on_board yes) (fields_autoplaced)
+    (property "Reference" "RV?" (id 0) (at 218.694 79.1015 0)
+      (effects (font (size 1.27 1.27)) (justify right))
+    )
+    (property "Value" "100k" (id 1) (at 218.694 81.8766 0)
+      (effects (font (size 1.27 1.27)) (justify right))
+    )
+    (property "Footprint" "" (id 2) (at 217.17 80.01 0)
+      (effects (font (size 1.27 1.27)) hide)
+    )
+    (property "Datasheet" "~" (id 3) (at 217.17 80.01 0)
+      (effects (font (size 1.27 1.27)) hide)
+    )
+    (pin "1")
+    (pin "2")
+    (pin "3")
   )
   (sheet_instances
@@
     )
     (path "/00000000-0000-0000-0000-00006156584c"
-      (reference "C1") (unit 1) (value "10n") (footprint "")
+      (reference "C1") (unit 1) (value "10nF") (footprint "")
     )
     (path "/00000000-0000-0000-0000-00006156678e"
-      (reference "C2") (unit 1) (value "1u") (footprint "")
+      (reference "C2") (unit 1) (value "1uF") (footprint "")
     )
     (path "/00000000-0000-0000-0000-00006150c7ad"
@@
       (reference "R18") (unit 1) (value "10k") (footprint "")
     )
-    (path "/00000000-0000-0000-0000-000061561e38"
-      (reference "RV1") (unit 1) (value "100k") (footprint "")
-    )
-    (path "/00000000-0000-0000-0000-000061563766"
-      (reference "RV2") (unit 1) (value "100k") (footprint "")
-    )
-  )
+    (path "/4280fd48-ab79-4594-b4bb-1546eb8e65b1"
+      (reference "RV?") (unit 1) (value "100k") (footprint "")
+    )
+    (path "/d838f757-590a-4fa3-8bcd-2f64ea9b3654"
+      (reference "RV?") (unit 1) (value "100k") (footprint "")
+    )
+  )
